Commit message: feature: Create f1tenth_gazebo package

File: src/f1tenth_gazebo/models/f1tenth/model.urdf (robot description, URDF)
Before this commit: robot f1tenth, 6 links, 5 joints
Links:
- added link link_steering_wheel, mass 0.2
Joints:
- removed joint joint_front_left_wheel
- removed joint joint_front_right_wheel
- added joint front_left_combined_joint: type continuous, parent link_chassis, child link_front_left_wheel, origin xyz=0 0 0 rpy=0.087 0 0, axis 0 1 0, limit effort=10000 velocity=1000
- added joint front_right_combined_joint: type continuous, parent link_chassis, child link_front_right_wheel, origin xyz=0 0 0 rpy=-0.087 0 0, axis 0 1 0, limit effort=10000 velocity=1000
- added joint joint_steering: type revolute, parent link_chassis, child link_steering_wheel, origin xyz=0.2 -0.17 0 rpy=0 0 0, axis 0 0 1, limit lower=-0.7 upper=0.7 effort=10000 velocity=1000
