Commit message: Remove robot folder and add custom plugin

File: src/f1tenth_description/urdf/f1tenth/model.urdf (robot description, URDF)
Before this commit: robot f1tenth, 7 links, 6 joints
Links:
- removed link link_steering_wheel
Joints:
- removed joint front_left_combined_joint
- removed joint front_right_combined_joint
- removed joint joint_steering
- added joint joint_front_left_wheel: type revolute, parent link_chassis, child link_front_left_wheel, origin xyz=0.2 -0.17 0 rpy=0 0 0, axis 0 0 1, limit lower=-0.7 upper=0.7 effort=10000 velocity=1000
- added joint joint_front_right_wheel: type revolute, parent link_chassis, child link_front_right_wheel, origin xyz=0.2 0.17 0 rpy=0 0 0, axis 0 0 1, limit lower=-0.7 upper=0.7 effort=10000 velocity=1000
